Commit message: Add joint to make camera oscillate in the demo

File: mujoco_ros2_control_demos/urdf/test_camera.xacro.urdf (robot description, URDF)
Before this commit: robot camera, 4 links, 3 joints
Joints:
- joint camera_joint: axis (none) -> 0 1 0; limit (none) -> lower=-0.5 upper=0.5 effort=1 velocity=1; type fixed -> revolute

Commit message: Initial support for depth data

File: mujoco_ros2_control_demos/urdf/test_camera.xacro.urdf (robot description, URDF)
Before this commit: robot camera, 4 links, 3 joints
Links:
- added link camera_optical_frame
Joints:
- added joint camera_optical_joint: type fixed, parent camera, child camera_optical_frame, origin xyz=0 0 0 rpy=-1.5708 0 -1.5708, axis 0 0 0
- joint camera_joint: axis 0 1 0 -> 0 0 1; origin xyz=0 0 1 rpy=0 0 0 -> xyz=0 0 1 rpy=0 1.5708 1.5708

Commit message: Add note and fix frame conventions for camera

File: mujoco_ros2_control_demos/urdf/test_camera.xacro.urdf (robot description, URDF)
Before this commit: robot camera, 5 links, 4 joints
Joints:
- joint camera_joint: axis 0 0 1 -> 0 1 0; limit lower=-0.5 upper=0.5 effort=1 velocity=1 -> lower=-0.5236 upper=0.5236 effort=1 velocity=1; origin xyz=0 0 1 rpy=0 1.5708 1.5708 -> xyz=0 0 1 rpy=0 0 0
- joint camera_optical_joint: origin xyz=0 0 0 rpy=-1.5708 0 -1.5708 -> xyz=0 0 0 rpy=3.14159 0 0
